Commit message: fixed bugs in transmission.Added gazebo plugin dep.

File: models/barrett_wam.transmission.xacro (robot description, xacro)
@@ -38,10 +38,10 @@
       </actuator>
     </transmission>
-    <transmission name="${prefix}/wrist_yaw_joint_trans">
+    <transmission name="${prefix}/wrist_yaw_trans">
       <type>transmission_interface/SimpleTransmission</type>
-      <joint name="${prefix}/wrist_yaw_joint_joint">
+      <joint name="${prefix}/wrist_yaw_joint">
         <hardwareInterface>PositionJointInterface</hardwareInterface>
       </joint>
-      <actuator name="${prefix}/wrist_yaw_joint_motor">
+      <actuator name="${prefix}/wrist_yaw_motor">
         <mechanicalReduction>1</mechanicalReduction>
       </actuator>

File: models/wam_top.urdf.xacro (robot description, xacro)
@@ -3,4 +3,5 @@
 <!-- Not needed for new Gazebo (http://gazebosim.org/tutorials/?tut=ros_urdf) -->
   <!-- xmlns:controller="http://playerstage.sourceforge.net/gazebo/xmlschema/#controller"> -->
+  <xacro:include filename="$(find barrett_model)/robots/common.gazebo.xacro" />
   <!-- Some macros used by the WAM urdf -->
   <xacro:include filename="$(find barrett_model)/models/common.urdf.xacro"/>
