Commit message: Added hand transmission

File: models/barrett_wam_hand.transmission.xacro (robot description, xacro)
@@ -1,65 +1,74 @@
 <?xml version="1.0"?>
 <robot xmlns:xacro="http://ros.org/wiki/xacro">
-  <xacro:macro name="wam_arm_transmission" params="prefix">
-    <transmission name="${prefix}/base_yaw_trans">
+  <xacro:macro name="wam_hand_transmission" params="prefix">
+    <transmission name="${prefix}/finger_1/prox_trans">
       <type>transmission_interface/SimpleTransmission</type>
-      <joint name="${prefix}/base_yaw_joint">
+      <joint name="${prefix}/finger_1/prox_joint">
         <hardwareInterface>PositionJointInterface</hardwareInterface>
       </joint>
-      <actuator name="${prefix}/base_yaw_motor">
+      <actuator name="${prefix}/finger_1/prox_motor">
         <mechanicalReduction>1</mechanicalReduction>
       </actuator>
     </transmission>
-    <transmission name="${prefix}/shoulder_pitch_trans">
+    <transmission name="${prefix}/finger_1/med_trans">
       <type>transmission_interface/SimpleTransmission</type>
-      <joint name="${prefix}/shoulder_pitch_joint">
+      <joint name="${prefix}/finger_1/med_joint">
         <hardwareInterface>PositionJointInterface</hardwareInterface>
       </joint>
-      <actuator name="${prefix}/shoulder_pitch_motor">
+      <actuator name="${prefix}/finger_1/med_motor">
         <mechanicalReduction>1</mechanicalReduction>
       </actuator>
     </transmission>
-    <transmission name="${prefix}/shoulder_yaw_trans">
+    <transmission name="${prefix}/finger_1/dist_trans">
       <type>transmission_interface/SimpleTransmission</type>
-      <joint name="${prefix}/shoulder_yaw_joint">
+      <joint name="${prefix}/finger_1/dist_joint">
         <hardwareInterface>PositionJointInterface</hardwareInterface>
       </joint>
-      <actuator name="${prefix}/shoulder_yaw_motor">
+      <actuator name="${prefix}/finger_1/dist_motor">
         <mechanicalReduction>1</mechanicalReduction>
       </actuator>
     </transmission>
-    <transmission name="${prefix}/elbow_pitch_trans">
+    <transmission name="${prefix}/finger_2/prox_trans">
       <type>transmission_interface/SimpleTransmission</type>
-      <joint name="${prefix}/elbow_pitch_joint">
+      <joint name="${prefix}/finger_2/prox_joint">
         <hardwareInterface>PositionJointInterface</hardwareInterface>
       </joint>
-      <actuator name="${prefix}/elbow_pitch_motor">
+      <actuator name="${prefix}/finger_2/prox_motor">
         <mechanicalReduction>1</mechanicalReduction>
       </actuator>
     </transmission>
-    <transmission name="${prefix}/wrist_yaw_trans">
+    <transmission name="${prefix}/finger_2/med_trans">
       <type>transmission_interface/SimpleTransmission</type>
-      <joint name="${prefix}/wrist_yaw_joint">
+      <joint name="${prefix}/finger_2/med_joint">
         <hardwareInterface>PositionJointInterface</hardwareInterface>
       </joint>
-      <actuator name="${prefix}/wrist_yaw_motor">
+      <actuator name="${prefix}/finger_2/med_motor">
         <mechanicalReduction>1</mechanicalReduction>
       </actuator>
     </transmission>
-    <transmission name="${prefix}/wrist_pitch_trans">
+    <transmission name="${prefix}/finger_2/dist_trans">
       <type>transmission_interface/SimpleTransmission</type>
-      <joint name="${prefix}/wrist_pitch_joint">
+      <joint name="${prefix}/finger_2/dist_joint">
         <hardwareInterface>PositionJointInterface</hardwareInterface>
       </joint>
-      <actuator name="${prefix}/wrist_pitch_motor">
+      <actuator name="${prefix}/finger_2/dist_motor">
         <mechanicalReduction>1</mechanicalReduction>
       </actuator>
     </transmission>
-    <transmission name="${prefix}/palm_yaw_trans">
+    <transmission name="${prefix}/finger_3/med_trans">
       <type>transmission_interface/SimpleTransmission</type>
-      <joint name="${prefix}/palm_yaw_joint">
+      <joint name="${prefix}/finger_3/med_joint">
         <hardwareInterface>PositionJointInterface</hardwareInterface>
       </joint>
-      <actuator name="${prefix}/palm_yaw_motor">
+      <actuator name="${prefix}/finger_3/med_motor">
+        <mechanicalReduction>1</mechanicalReduction>
+      </actuator>
+    </transmission>
+    <transmission name="${prefix}/finger_3/dist_trans">
+      <type>transmission_interface/SimpleTransmission</type>
+      <joint name="${prefix}/finger_3/dist_joint">
+        <hardwareInterface>PositionJointInterface</hardwareInterface>
+      </joint>
+      <actuator name="${prefix}/finger_3/dist_motor">
         <mechanicalReduction>1</mechanicalReduction>
       </actuator>

File: models/hand.urdf.xacro (robot description, xacro)
@@ -1,3 +1,4 @@
 <robot xmlns:xacro="http://www.ros.org/wiki/xacro">
+  <xacro:include filename="$(find barrett_model)/models/barrett_wam_hand.transmission.xacro" />
   <xacro:include filename="$(find barrett_model)/models/common.urdf.xacro"/>
   <!-- link properties -->
@@ -34,4 +35,5 @@
     <xacro:bhand_finger_2 prefix="${prefix}" primitive="${primitive}"/>
     <xacro:bhand_finger_3 prefix="${prefix}" primitive="${primitive}"/>
+    <xacro:wam_hand_transmission prefix="${prefix}" />
     <!-- don't use the gazebo gripper plugin, just slows down the sim -->
     <xacro:if value="false">

File: robots/common.gazebo.xacro (robot description, xacro)
@@ -3,5 +3,5 @@
   <gazebo>
     <plugin name="ros_control" filename="libgazebo_ros_control.so">
-      <robotNamespace>/barrett_wam</robotNamespace>
+      <robotNamespace>/wam</robotNamespace>
       <!--robotSimType>gazebo_ros_control/DefaultRobotHWSim</robotSimType-->
     </plugin>
