Commit message: added effort transmission. Use "effort_control" boolean arg when calling "wam_7dof" xacro.

File: models/arm.urdf.xacro (robot description, xacro)
@@ -24,12 +24,12 @@
 -->
 <robot xmlns:xacro="http://www.ros.org/wiki/xacro">
-  <xacro:include filename="$(find barrett_model)/models/barrett_wam.transmission.xacro" />
   <xacro:include filename="$(find barrett_model)/models/common.urdf.xacro"/>
   <xacro:include filename="$(find barrett_model)/models/components.urdf.xacro"/>
-  <xacro:macro name="wam_7dof" params="prefix parent_link xyz rpy">
+  <xacro:macro name="wam_7dof" params="prefix effort_control parent_link xyz rpy">
+    <xacro:include filename="$(find barrett_model)/models/barrett_wam.transmission.xacro" />
     <xacro:wam prefix="${prefix}" parent_link="${parent_link}" xyz="${xyz}" rpy="${rpy}"/>
     <xacro:wam_wrist prefix="${prefix}"/>
     <xacro:wam_wrist_palm_stump prefix="${prefix}"/>
-    <xacro:wam_arm_transmission prefix="${prefix}" />
+    <xacro:wam_arm_transmission prefix="${prefix}" effort="${effort_control}" />
   </xacro:macro>
   <xacro:macro name="wam_4dof" params="prefix parent_link xyz rpy">

File: models/barrett_wam.transmission.xacro (robot description, xacro)
@@ -1,9 +1,14 @@
 <?xml version="1.0"?>
 <robot xmlns:xacro="http://ros.org/wiki/xacro">
-  <xacro:macro name="wam_arm_transmission" params="prefix">
+  <xacro:macro name="wam_arm_transmission" params="prefix effort">
     <transmission name="${prefix}/base_yaw_trans">
       <type>transmission_interface/SimpleTransmission</type>
       <joint name="${prefix}/base_yaw_joint">
-        <hardwareInterface>PositionJointInterface</hardwareInterface>
+        <xacro:if value="${effort}">
+          <hardwareInterface>hardware_interface/EffortJointInterface</hardwareInterface>
+        </xacro:if>
+        <xacro:unless value="${effort}">
+          <hardwareInterface>hardware_interface/PositionJointInterface</hardwareInterface>
+        </xacro:unless>
       </joint>
       <actuator name="${prefix}/base_yaw_motor">
@@ -14,5 +19,10 @@
       <type>transmission_interface/SimpleTransmission</type>
       <joint name="${prefix}/shoulder_pitch_joint">
-        <hardwareInterface>PositionJointInterface</hardwareInterface>
+        <xacro:if value="${effort}">
+          <hardwareInterface>hardware_interface/EffortJointInterface</hardwareInterface>
+        </xacro:if>
+        <xacro:unless value="${effort}">
+          <hardwareInterface>hardware_interface/PositionJointInterface</hardwareInterface>
+        </xacro:unless>
       </joint>
       <actuator name="${prefix}/shoulder_pitch_motor">
@@ -23,5 +33,10 @@
       <type>transmission_interface/SimpleTransmission</type>
       <joint name="${prefix}/shoulder_yaw_joint">
-        <hardwareInterface>PositionJointInterface</hardwareInterface>
+        <xacro:if value="${effort}">
+          <hardwareInterface>hardware_interface/EffortJointInterface</hardwareInterface>
+        </xacro:if>
+        <xacro:unless value="${effort}">
+          <hardwareInterface>hardware_interface/PositionJointInterface</hardwareInterface>
+        </xacro:unless>
       </joint>
       <actuator name="${prefix}/shoulder_yaw_motor">
@@ -32,5 +47,10 @@
       <type>transmission_interface/SimpleTransmission</type>
       <joint name="${prefix}/elbow_pitch_joint">
-        <hardwareInterface>PositionJointInterface</hardwareInterface>
+        <xacro:if value="${effort}">
+          <hardwareInterface>hardware_interface/EffortJointInterface</hardwareInterface>
+        </xacro:if>
+        <xacro:unless value="${effort}">
+          <hardwareInterface>hardware_interface/PositionJointInterface</hardwareInterface>
+        </xacro:unless>
       </joint>
       <actuator name="${prefix}/elbow_pitch_motor">
@@ -41,5 +61,10 @@
       <type>transmission_interface/SimpleTransmission</type>
       <joint name="${prefix}/wrist_yaw_joint">
-        <hardwareInterface>PositionJointInterface</hardwareInterface>
+        <xacro:if value="${effort}">
+          <hardwareInterface>hardware_interface/EffortJointInterface</hardwareInterface>
+        </xacro:if>
+        <xacro:unless value="${effort}">
+          <hardwareInterface>hardware_interface/PositionJointInterface</hardwareInterface>
+        </xacro:unless>
       </joint>
       <actuator name="${prefix}/wrist_yaw_motor">
@@ -50,5 +75,10 @@
       <type>transmission_interface/SimpleTransmission</type>
       <joint name="${prefix}/wrist_pitch_joint">
-        <hardwareInterface>PositionJointInterface</hardwareInterface>
+        <xacro:if value="${effort}">
+          <hardwareInterface>hardware_interface/EffortJointInterface</hardwareInterface>
+        </xacro:if>
+        <xacro:unless value="${effort}">
+          <hardwareInterface>hardware_interface/PositionJointInterface</hardwareInterface>
+        </xacro:unless>
       </joint>
       <actuator name="${prefix}/wrist_pitch_motor">
@@ -59,5 +89,10 @@
       <type>transmission_interface/SimpleTransmission</type>
       <joint name="${prefix}/palm_yaw_joint">
-        <hardwareInterface>PositionJointInterface</hardwareInterface>
+        <xacro:if value="${effort}">
+          <hardwareInterface>hardware_interface/EffortJointInterface</hardwareInterface>
+        </xacro:if>
+        <xacro:unless value="${effort}">
+          <hardwareInterface>hardware_interface/PositionJointInterface</hardwareInterface>
+        </xacro:unless>
       </joint>
       <actuator name="${prefix}/palm_yaw_motor">

File: models/barrett_wam_hand.transmission.xacro (robot description, xacro)
@@ -5,5 +5,5 @@
       <type>transmission_interface/SimpleTransmission</type>
       <joint name="${prefix}/finger_1/prox_joint">
-        <hardwareInterface>PositionJointInterface</hardwareInterface>
+        <hardwareInterface>hardware_interface/PositionJointInterface</hardwareInterface>
       </joint>
       <actuator name="${prefix}/finger_1/prox_motor">
@@ -14,5 +14,5 @@
       <type>transmission_interface/SimpleTransmission</type>
       <joint name="${prefix}/finger_1/med_joint">
-        <hardwareInterface>PositionJointInterface</hardwareInterface>
+        <hardwareInterface>hardware_interface/PositionJointInterface</hardwareInterface>
       </joint>
       <actuator name="${prefix}/finger_1/med_motor">
@@ -23,5 +23,5 @@
       <type>transmission_interface/SimpleTransmission</type>
       <joint name="${prefix}/finger_1/dist_joint">
-        <hardwareInterface>PositionJointInterface</hardwareInterface>
+        <hardwareInterface>hardware_interface/PositionJointInterface</hardwareInterface>
       </joint>
       <actuator name="${prefix}/finger_1/dist_motor">
@@ -32,5 +32,5 @@
       <type>transmission_interface/SimpleTransmission</type>
       <joint name="${prefix}/finger_2/prox_joint">
-        <hardwareInterface>PositionJointInterface</hardwareInterface>
+        <hardwareInterface>hardware_interface/PositionJointInterface</hardwareInterface>
       </joint>
       <actuator name="${prefix}/finger_2/prox_motor">
@@ -41,5 +41,5 @@
       <type>transmission_interface/SimpleTransmission</type>
       <joint name="${prefix}/finger_2/med_joint">
-        <hardwareInterface>PositionJointInterface</hardwareInterface>
+        <hardwareInterface>hardware_interface/PositionJointInterface</hardwareInterface>
       </joint>
       <actuator name="${prefix}/finger_2/med_motor">
@@ -50,5 +50,5 @@
       <type>transmission_interface/SimpleTransmission</type>
       <joint name="${prefix}/finger_2/dist_joint">
-        <hardwareInterface>PositionJointInterface</hardwareInterface>
+        <hardwareInterface>hardware_interface/PositionJointInterface</hardwareInterface>
       </joint>
       <actuator name="${prefix}/finger_2/dist_motor">
@@ -59,5 +59,5 @@
       <type>transmission_interface/SimpleTransmission</type>
       <joint name="${prefix}/finger_3/med_joint">
-        <hardwareInterface>PositionJointInterface</hardwareInterface>
+        <hardwareInterface>hardware_interface/PositionJointInterface</hardwareInterface>
       </joint>
       <actuator name="${prefix}/finger_3/med_motor">
@@ -68,5 +68,5 @@
       <type>transmission_interface/SimpleTransmission</type>
       <joint name="${prefix}/finger_3/dist_joint">
-        <hardwareInterface>PositionJointInterface</hardwareInterface>
+        <hardwareInterface>hardware_interface/PositionJointInterface</hardwareInterface>
       </joint>
       <actuator name="${prefix}/finger_3/dist_motor">

File: robots/wam_7dof_wam_bhand.urdf.xacro (robot description, xacro)
@@ -5,5 +5,5 @@
   <!-- Root link is in the world frame-->
   <link name = "world"/>
-  <xacro:wam_7dof prefix="wam" parent_link="world" xyz="0.02 0.46 1" rpy="0 0 0" />
+  <xacro:wam_7dof prefix="wam" effort_control="true" parent_link="world" xyz="0.02 0.46 1" rpy="0 0 0" />
   <xacro:bhand prefix="wam/bhand" parent_link="wam/wrist_palm_link" xyz="0 0 0.06" rpy="0 0 ${PI}" primitive="true"/>
 </robot>

Commit message: Velocity transmission and joint traj. control. Refactored launchfiles for readability.

File: models/arm.urdf.xacro (robot description, xacro)
@@ -26,10 +26,10 @@
   <xacro:include filename="$(find barrett_model)/models/common.urdf.xacro"/>
   <xacro:include filename="$(find barrett_model)/models/components.urdf.xacro"/>
-  <xacro:macro name="wam_7dof" params="prefix effort_control parent_link xyz rpy">
-    <xacro:include filename="$(find barrett_model)/models/barrett_wam.transmission.xacro" />
+  <xacro:macro name="wam_7dof" params="prefix parent_link xyz rpy">
+    <xacro:include filename="$(find barrett_model)/models/barrett_wam.transmission_$(arg ctrl_mode).xacro" />
     <xacro:wam prefix="${prefix}" parent_link="${parent_link}" xyz="${xyz}" rpy="${rpy}"/>
     <xacro:wam_wrist prefix="${prefix}"/>
     <xacro:wam_wrist_palm_stump prefix="${prefix}"/>
-    <xacro:wam_arm_transmission prefix="${prefix}" effort="${effort_control}" />
+    <xacro:wam_arm_transmission prefix="${prefix}"/>
   </xacro:macro>
   <xacro:macro name="wam_4dof" params="prefix parent_link xyz rpy">

File: models/barrett_wam.transmission_effort.xacro (robot description, xacro)
@@ -1,14 +1,9 @@
 <?xml version="1.0"?>
 <robot xmlns:xacro="http://ros.org/wiki/xacro">
-  <xacro:macro name="wam_arm_transmission" params="prefix effort">
+  <xacro:macro name="wam_arm_transmission" params="prefix">
     <transmission name="${prefix}/base_yaw_trans">
       <type>transmission_interface/SimpleTransmission</type>
       <joint name="${prefix}/base_yaw_joint">
-        <xacro:if value="${effort}">
-          <hardwareInterface>hardware_interface/EffortJointInterface</hardwareInterface>
-        </xacro:if>
-        <xacro:unless value="${effort}">
-          <hardwareInterface>hardware_interface/PositionJointInterface</hardwareInterface>
-        </xacro:unless>
+        <hardwareInterface>hardware_interface/EffortJointInterface</hardwareInterface>
       </joint>
       <actuator name="${prefix}/base_yaw_motor">
@@ -19,10 +14,5 @@
       <type>transmission_interface/SimpleTransmission</type>
       <joint name="${prefix}/shoulder_pitch_joint">
-        <xacro:if value="${effort}">
-          <hardwareInterface>hardware_interface/EffortJointInterface</hardwareInterface>
-        </xacro:if>
-        <xacro:unless value="${effort}">
-          <hardwareInterface>hardware_interface/PositionJointInterface</hardwareInterface>
-        </xacro:unless>
+        <hardwareInterface>hardware_interface/EffortJointInterface</hardwareInterface>
       </joint>
       <actuator name="${prefix}/shoulder_pitch_motor">
@@ -33,10 +23,5 @@
       <type>transmission_interface/SimpleTransmission</type>
       <joint name="${prefix}/shoulder_yaw_joint">
-        <xacro:if value="${effort}">
-          <hardwareInterface>hardware_interface/EffortJointInterface</hardwareInterface>
-        </xacro:if>
-        <xacro:unless value="${effort}">
-          <hardwareInterface>hardware_interface/PositionJointInterface</hardwareInterface>
-        </xacro:unless>
+        <hardwareInterface>hardware_interface/EffortJointInterface</hardwareInterface>
       </joint>
       <actuator name="${prefix}/shoulder_yaw_motor">
@@ -47,10 +32,5 @@
       <type>transmission_interface/SimpleTransmission</type>
       <joint name="${prefix}/elbow_pitch_joint">
-        <xacro:if value="${effort}">
-          <hardwareInterface>hardware_interface/EffortJointInterface</hardwareInterface>
-        </xacro:if>
-        <xacro:unless value="${effort}">
-          <hardwareInterface>hardware_interface/PositionJointInterface</hardwareInterface>
-        </xacro:unless>
+        <hardwareInterface>hardware_interface/EffortJointInterface</hardwareInterface>
       </joint>
       <actuator name="${prefix}/elbow_pitch_motor">
@@ -61,10 +41,5 @@
       <type>transmission_interface/SimpleTransmission</type>
       <joint name="${prefix}/wrist_yaw_joint">
-        <xacro:if value="${effort}">
-          <hardwareInterface>hardware_interface/EffortJointInterface</hardwareInterface>
-        </xacro:if>
-        <xacro:unless value="${effort}">
-          <hardwareInterface>hardware_interface/PositionJointInterface</hardwareInterface>
-        </xacro:unless>
+        <hardwareInterface>hardware_interface/EffortJointInterface</hardwareInterface>
       </joint>
       <actuator name="${prefix}/wrist_yaw_motor">
@@ -75,10 +50,5 @@
       <type>transmission_interface/SimpleTransmission</type>
       <joint name="${prefix}/wrist_pitch_joint">
-        <xacro:if value="${effort}">
-          <hardwareInterface>hardware_interface/EffortJointInterface</hardwareInterface>
-        </xacro:if>
-        <xacro:unless value="${effort}">
-          <hardwareInterface>hardware_interface/PositionJointInterface</hardwareInterface>
-        </xacro:unless>
+        <hardwareInterface>hardware_interface/EffortJointInterface</hardwareInterface>
       </joint>
       <actuator name="${prefix}/wrist_pitch_motor">
@@ -89,10 +59,5 @@
       <type>transmission_interface/SimpleTransmission</type>
       <joint name="${prefix}/palm_yaw_joint">
-        <xacro:if value="${effort}">
-          <hardwareInterface>hardware_interface/EffortJointInterface</hardwareInterface>
-        </xacro:if>
-        <xacro:unless value="${effort}">
-          <hardwareInterface>hardware_interface/PositionJointInterface</hardwareInterface>
-        </xacro:unless>
+        <hardwareInterface>hardware_interface/EffortJointInterface</hardwareInterface>
       </joint>
       <actuator name="${prefix}/palm_yaw_motor">

File: robots/wam_7dof_wam_bhand.urdf.xacro (robot description, xacro)
@@ -1,9 +1,10 @@
 <robot name="wam"
   xmlns:xacro="http://www.ros.org/wiki/xacro">
+  <xacro:arg name="ctrl_mode" default="position"/>
   <!-- Include all the WAM stuff -->
   <include filename="$(find barrett_model)/models/wam_top.urdf.xacro"/>
   <!-- Root link is in the world frame-->
   <link name = "world"/>
-  <xacro:wam_7dof prefix="wam" effort_control="true" parent_link="world" xyz="0.02 0.46 1" rpy="0 0 0" />
+  <xacro:wam_7dof prefix="wam" parent_link="world" xyz="0.02 0.46 1" rpy="0 0 0" />
   <xacro:bhand prefix="wam/bhand" parent_link="wam/wrist_palm_link" xyz="0 0 0.06" rpy="0 0 ${PI}" primitive="true"/>
 </robot>
