Commit message: simplified setting ofjoint velocity limits

File: models/components.urdf.xacro (robot description, xacro)
@@ -27,4 +27,6 @@
   <xacro:include filename="$(find barrett_model)/models/common.urdf.xacro"/>
   <xacro:property name="b" value="0.5"/>
+  <xacro:property name="vel_lim" value="10.0"/>
+  <!-- <xacro:property name="vel_lim" value="2.0"/> -->
   <!-- Upper arm macros -->
   <xacro:macro name="wam_base" params="prefix parent_link xyz rpy">
@@ -67,5 +69,5 @@
       <origin xyz="0 0 0.346" rpy="0 0 0"/>
       <axis xyz="0 0 1"/>
-      <limit effort="60" lower="-2.6" upper="2.6" velocity="2.0"/>
+      <limit effort="60" lower="-2.6" upper="2.6" velocity="${vel_lim}"/>
       <dynamics damping="${1.8*b}" friction="0"/>
     </joint>
@@ -106,5 +108,5 @@
       <origin xyz="0 0 0" rpy="${-PI/2} 0 0"/>
       <axis xyz="0 0 1"/>
-      <limit effort="60" lower="-1.985" upper="1.985" velocity="2.0"/>
+      <limit effort="60" lower="-1.985" upper="1.985" velocity="${vel_lim}"/>
       <dynamics damping="${0.5*b}" friction="0"/>
     </joint>
@@ -145,5 +147,5 @@
       <origin xyz="0 0 0" rpy="${PI/2} 0 0"/>
       <axis xyz="0 0 1"/>
-      <limit effort="45" lower="-2.8" upper="2.8" velocity="2.0"/>
+      <limit effort="45" lower="-2.8" upper="2.8" velocity="${vel_lim}"/>
       <dynamics damping="${1.5*b}" friction="0"/>
     </joint>
@@ -185,5 +187,5 @@
       <origin xyz="0.045 0 0.55" rpy="${-PI/2} 0 0"/>
       <axis xyz="0 0 1"/>
-      <limit effort="30" lower="-0.9" upper="${PI}" velocity="2.00"/>
+      <limit effort="30" lower="-0.9" upper="${PI}" velocity="${vel_lim}"/>
       <dynamics damping="${0.8*b}" friction="0"/>
     </joint>
@@ -239,5 +241,5 @@
       <origin xyz="-0.045 -0.3 0" rpy="${PI/2} 0 0"/>
       <axis xyz="0 0 1"/>
-      <limit effort="10" lower="-4.55" upper="1.25" velocity="2.0"/>
+      <limit effort="10" lower="-4.55" upper="1.25" velocity="${vel_lim}"/>
       <dynamics damping="${0.5*b}" friction="0"/>
     </joint>
@@ -279,5 +281,5 @@
       <origin xyz="0 0 0" rpy="${-PI/2} 0 0"/>
       <axis xyz="0 0 1"/>
-      <limit effort="10" lower="-1.5707" upper="1.5707" velocity="2.00"/>
+      <limit effort="10" lower="-1.5707" upper="1.5707" velocity="${vel_lim}"/>
       <dynamics damping="${0.1*b}" friction="0"/>
     </joint>
@@ -319,5 +321,5 @@
       <origin xyz="0 0 0" rpy="${PI/2} 0 0"/>
       <axis xyz="0 0 1"/>
-      <limit effort="10" lower="-3.0" upper="3.0" velocity="2.00"/><!-- 2.95 is a limit taken in from 3 due to saftey and differences between arms. -->
+      <limit effort="10" lower="-3.0" upper="3.0" velocity="${vel_lim}"/><!-- 2.95 is a limit taken in from 3 due to saftey and differences between arms. -->
       <dynamics damping="${0.3*b}" friction="0"/>
     </joint>
@@ -483,5 +485,5 @@
       <origin xyz="0.045 0 0.55" rpy="${-PI/2} 0 0"/>
       <axis xyz="0 0 1"/>
-      <limit effort="15" lower="-0.9" upper="${PI}" velocity="2.0"/>
+      <limit effort="15" lower="-0.9" upper="${PI}" velocity="${vel_lim}"/>
       <dynamics damping="${0.1*b}" friction="0"/>
     </joint>
