Commit message: rotation offset for FT frame

File: gtrll/wam_7dof_ft_ball.urdf (robot description, URDF)
Before this commit: robot wam, 12 links, 11 joints
Links:
- removed link world
Joints:
- removed joint wam/elbow_pitch_joint
- removed joint wam/palm_yaw_joint
- removed joint wam/shoulder_yaw_joint
- removed joint wam/wam_fixed_joint
- removed joint wam/wam_j2
- removed joint wam/wrist_pitch_joint
- removed joint wam/wrist_yaw_joint
- added joint wam_j2: type revolute, parent wam/shoulder_yaw_link, child wam/shoulder_pitch_link, origin xyz=0 0 0 rpy=-1.57079632679 0 0, axis 0 0 1, limit lower=-1.985 upper=1.985 effort=60 velocity=2.0
- added joint wam_j3: type revolute, parent wam/shoulder_pitch_link, child wam/upper_arm_link, origin xyz=0 0 0 rpy=1.57079632679 0 0, axis 0 0 1, limit lower=-2.8 upper=2.8 effort=45 velocity=2.0
- added joint wam_j4: type revolute, parent wam/upper_arm_link, child wam/forearm_link, origin xyz=0.045 0 0.55 rpy=-1.57079632679 0 0, axis 0 0 1, limit lower=-0.9 upper=3.14159265359 effort=30 velocity=2.00
- added joint wam_j5: type revolute, parent wam/forearm_link, child wam/wrist_yaw_link, origin xyz=-0.045 -0.3 0 rpy=1.57079632679 0 0, axis 0 0 1, limit lower=-4.55 upper=1.25 effort=10 velocity=2.0
- added joint wam_j6: type revolute, parent wam/wrist_yaw_link, child wam/wrist_pitch_link, origin xyz=0 0 0 rpy=-1.57079632679 0 0, axis 0 0 1, limit lower=-1.5707 upper=1.5707 effort=10 velocity=2.00
- added joint wam_j7: type revolute, parent wam/wrist_pitch_link, child wam/wrist_palm_link, origin xyz=0 0 0 rpy=1.57079632679 0 0, axis 0 0 1, limit lower=-3.0 upper=3.0 effort=10 velocity=2.00
- joint wam/ft_sensor_joint: origin xyz=0 0 0.0673 rpy=0 0 0 -> xyz=0 0 0.0673 rpy=0 0 1.570796

Commit message: changed ft_sensor_link origin

File: gtrll/wam_7dof_ft_ball.urdf (robot description, URDF)
Before this commit: robot wam, 11 links, 10 joints
Joints:
- joint wam/ft_sensor_joint: origin xyz=0 0 0.0673 rpy=0 0 1.570796 -> xyz=0 0 0.0673 rpy=0 0 0.0
